File: pcb/src/lornode.kicad_pcb (KiCad board)
At the start: 2 copper layers, 43.4 x 73.7 mm, 69 parts, among them J1 TYPE-C-31-M-12, J2 Breakout Right, J3 Breakout Left, J4 BATT_IN, J6 CHG_IN, J7 Breakout LoRA, Q1 YJL2301G, Q2 FS8205A, Q3 YJL2102W, Q4 YJL2102W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

Commit message: v2 minor updates
Other:
- board text added: "5V_I"
- board text removed: "5V"
